Commit message: proje init

File: src/my_robot_description/urdf/common_properties.xacro (robot description, xacro)
@@ -3,4 +3,10 @@
     <material name="blue">
         <color rgba="0 0 0.5 1" />
+    </material>
+    <material name="black">
+        <color rgba="0 0 0 1" />
+    </material>
+    <material name="red">
+        <color rgba="1 0 0 1" />
     </material>
     <material name="grey">

File: src/my_robot_description/urdf/mobile_base.xacro (robot description, xacro)
@@ -1,9 +1,14 @@
 <?xml version="1.0"?>
 <robot xmlns:xacro="http://www.ros.org/wiki/xacro">
-    <xacro:property name="base_length"  value="0.6"/>
-    <xacro:property name="base_width"  value="0.4"/>
-    <xacro:property name="base_height"  value="0.2"/>
-    <xacro:property name="wheel_radius"  value="0.1"/>
-    <xacro:property name="wheel_length"  value="0.05"/>
+    <xacro:property name="base_length"  value="2.5"/>
+    <xacro:property name="base_width"  value="1.5"/>
+    <xacro:property name="base_height"  value="1"/>
+    <xacro:property name="wheel_radius"  value="0.4"/>
+    <xacro:property name="wheel_length"  value="0.20"/>
+    <xacro:property name="gps_length" value="0.1"/>
+    <xacro:property name="gps_width" value="0.1"/>
+    <xacro:property name="gps_height" value="0.05"/>
+    <xacro:property name="dif_length" value="0.05"/>
+    <xacro:property name="dif_radius" value="0.02"/>
     <link name="base_footprint" />
     <link name="base_link">
@@ -13,71 +18,82 @@
             </geometry>
             <origin xyz="0 0 ${base_height / 2.0}" rpy="0 0 0" />
-            <material name="blue" />
-            <xacro:box_inertia m="5.0" l="${2*base_length}" w="${2*base_width}" h="${2*base_height}"
-                                xyz="0 0 ${base_height / 2.0}" rpy="0 0 0" />
+            <material name="red" />
         </visual>
         <collision>
             <geometry>
-                <box size="${base_length} ${base_width} ${base_height}" />
+                <box size="${base_length} ${base_width} ${base_height}"/>
             </geometry>
             <origin xyz="0 0 ${base_height / 2.0}" rpy="0 0 0" />
         </collision>
+        <xacro:box_inertia m="5.0" l="${2*base_length}" w="${2*base_width}" h="${2*base_height}"
+                                xyz="0 0 ${base_height / 2.0}" rpy="0 0 0" />
     </link>
-    <xacro:macro name="wheel_link" params="prefix">
+    <!-- SAĞ-SOL TEKER DİFERANSİYEL -->
+    <xacro:macro name="dif_link" params="prefix">
+        <link name="${prefix}_front_dif">
+            <visual>
+                <geometry>
+                    <cylinder length="${dif_length}" radius="${dif_radius}"/>
+                </geometry>
+                <origin xyz= "0 0 0" rpy="0 0 0"/>
+                <material name="black"/>
+            </visual>
+            <collision>
+                <geometry>
+                    <cylinder length="${dif_length}" radius="${dif_radius}"/>
+                </geometry>
+                <origin xyz= "0 0 0" rpy="0 0 0"/>
+            </collision>
+            <xacro:cylinder_inertia m="1" r="${2*dif_radius}" l="${2*dif_length}"
+                            xyz="0 0 0" rpy="0 0 0" />
+        </link>
+    </xacro:macro>
+    <xacro:dif_link prefix="right"/>
+    <xacro:dif_link prefix="left"/>
+    <xacro:macro name="wheel_link" params="prefix radius_ length_ z_offset">
         <link name="${prefix}_wheel_link">
             <visual>
                 <geometry>
-                    <cylinder radius="${wheel_radius}" length="${wheel_length}" />
+                    <cylinder radius="${radius_}" length="${length_}" />
                 </geometry>
-                <origin xyz="0 0 0" rpy="${pi/2.0} 0 0" />
-                <material name="grey" />
+                <origin xyz="0 0 ${z_offset/2.0}" rpy="0 0 0" />
+                <material name="black" />
             </visual>
             <collision>
                 <geometry>
-                    <cylinder radius="${wheel_radius}" length="${wheel_length}" />
+                    <cylinder radius="${radius_}" length="${length_}" />
                 </geometry>
-                <origin xyz="0 0 0" rpy="${pi/2.0} 0 0" />
-        </collision>
-            <xacro:cylinder_inertia m="1.0" r="${2*wheel_radius}" l="${2*wheel_length}"
-                    xyz="0 0 0" rpy="${pi/2.0} 0 0" />
+                <origin xyz="0 0 ${z_offset/2.0}" rpy="0 0 0" />
+            </collision>
+            <xacro:cylinder_inertia m="1.0" r="${2*radius_}" l="${2*length_}"
+                    xyz="0 0 ${z_offset/2.0}" rpy="0 0 0" />
         </link>
     </xacro:macro>
-    <xacro:wheel_link prefix="right"/>
-    <xacro:wheel_link prefix="left"/>
-    <!-- <link name="right_wheel_link">
+    <xacro:wheel_link prefix="right_front" radius_="${wheel_radius}" length_="${wheel_length}"  z_offset="0"/>
+    <xacro:wheel_link prefix="left_front" radius_="${wheel_radius}" length_="${wheel_length}" z_offset="0"/>
+    <xacro:wheel_link prefix="right_back" radius_="${wheel_radius}" length_="${wheel_length}"  z_offset="${wheel_length}"/>
+    <xacro:wheel_link prefix="left_back" radius_="${wheel_radius}" length_="${wheel_length}" z_offset="${-wheel_length}"/>
+    <!-- <link name="steering_wheel_link">
         <visual>
             <geometry>
-                <cylinder radius="${wheel_radius}" length="${wheel_length}" />
+                <cylinder length="0.05" radius="0.2"/>
             </geometry>
-            <origin xyz="0 0 0" rpy="${pi/2.0} 0 0" />
-            <material name="grey" />
-        </visual>
-    </link>
-    <link name="left_wheel_link">
-        <visual>
-            <geometry>
-                <cylinder radius="${wheel_radius}" length="${wheel_length}" />
-            </geometry>
-            <origin xyz="0 0 0" rpy="${pi/2.0} 0 0" />
-            <material name="grey" />
-        </visual>
-    </link> -->
-    <link name="caster_wheel_link">
-        <visual>
-            <geometry>
-                <sphere radius="${wheel_radius/2.0}" />
-            </geometry>
-            <origin xyz="0 0 0" rpy="0 0 0" />
-            <material name="grey" />
+            <material name="grey"/>
         </visual>
         <collision>
             <geometry>
-                <sphere radius="${wheel_radius/2.0}" />
+                <cylinder length="0.05" radius="0.2"/>
             </geometry>
-            <origin xyz="0 0 0" rpy="0 0 0" />
         </collision>
-        <xacro:sphere_inertia m="0.5" r="${2*wheel_radius/2.0}"
-                    xyz="0 0 0" rpy="0 0 0" />
-    </link>
+        <inertial>
+            <mass value="0.5"/>
+            <inertia ixx="0.001" ixy="0" ixz="0" iyy="0.001" iyz="0" izz="0.001"/>
+        </inertial>
+    </link> -->
+    <joint name="base_footprint_joint" type="fixed">
+        <parent link="odom"/>
+        <child link="base_footprint"/>
+        <origin rpy="0 0 0" xyz="0 0 0"/>
+    </joint>
     <joint name="base_joint" type="fixed">
         <parent link="base_footprint" />
@@ -85,20 +101,54 @@
         <origin xyz="0 0 ${wheel_radius}" rpy="0 0 0"/>
     </joint>
-    <joint name="base_right_wheel_joint" type="continuous">
+    <joint name="left_front_dif_joint" type="revolute">
         <parent link="base_link" />
-        <child link="right_wheel_link" />
-        <origin xyz="${-base_length / 4.0} ${-(base_height + (wheel_length/2))} 0" rpy="0 0 0" />
+        <child link="left_front_dif" />
+        <origin xyz="${base_length / 4.0} ${(base_width/2.0) + (wheel_length/2.0)} 0" rpy="${pi/2.0} 0 0" />
         <axis xyz="0 1 0" />
+        <limit effort="100" velocity="1" lower="-1" upper="1"/>
+        <dynamics damping="0.0" friction="0.0"/>
     </joint>
-    <joint name="base_left_wheel_joint" type="continuous">
+    <joint name="right_front_dif_joint" type="revolute">
         <parent link="base_link" />
-        <child link="left_wheel_link" />
-        <origin xyz="${-base_length / 4.0} ${base_height + (wheel_length/2)} 0" rpy="0 0 0" />
+        <child link="right_front_dif" />
+        <origin xyz="${base_length / 4.0} ${-((base_width/2.0) + (wheel_length/2.0))} 0" rpy="${pi/2.0} 0 0" />
         <axis xyz="0 1 0" />
+        <limit effort="100" velocity="1" lower="-1" upper="1"/>
+        <dynamics damping="0.0" friction="0.0"/>
     </joint>
-    <joint name="base_caster_wheel_joint" type="fixed">
+    <joint name="left_back_wheel_joint" type="continuous">
         <parent link="base_link" />
-        <child link="caster_wheel_link" />
-        <origin xyz="${base_length / 3.0} 0 ${-wheel_radius/2.0}" rpy="0 0 0" />
+        <child link="left_back_wheel_link" />
+        <origin xyz="${-base_length / 4.0} ${base_width/2.0} 0" rpy="${pi/2.0} 0 0" />
+        <axis xyz="0 0 -1" />
     </joint>
+    <joint name="right_back_wheel_joint" type="continuous">
+        <parent link="base_link" />
+        <child link="right_back_wheel_link" />
+        <origin xyz="${-base_length / 4.0} ${-base_width/2.0} 0" rpy="${pi/2.0} 0 0" />
+        <axis xyz="0 0 -1" />
+    </joint>
+    <joint name="left_front_dif_wheel_joint" type="continuous">
+        <parent link="left_front_dif" />
+        <child link="left_front_wheel_link"/>
+        <origin xyz="0 0 0" rpy="0 0 0"/>
+        <axis xyz="0 0 -1" />
+        <dynamics damping="0.0" friction="0.0"/>
+        <limit effort="100" velocity="100"/>
+    </joint>
+    <joint name="right_front_dif_wheel_joint" type="continuous">
+        <parent link="right_front_dif" />
+        <child link="right_front_wheel_link"/>
+        <origin xyz="0 0 0" rpy="0 0 0"/>
+        <axis xyz="0 0 -1" />
+        <dynamics damping="0.0" friction="0.0"/>
+        <limit effort="100" velocity="100"/>
+    </joint>
+<!--
+    <joint name="steering_wheel_joint" type="continuous">
+        <parent link="base_link" />
+        <child link="steering_wheel_link" />
+        <origin xyz="0 0 0" rpy="0 0 0" />
+        <axis xyz="0 0 1" />
+    </joint> -->
 </robot>

File: src/my_robot_description/urdf/mobile_base_gazebo.xacro (robot description, xacro)
@@ -2,39 +2,58 @@
 <robot xmlns:xacro="http://www.ros.org/wiki/xacro">
     <gazebo reference="base_link">
-        <material>Gazebo/Blue</material>
+        <material>Gazebo/Red</material>
     </gazebo>
-    <gazebo reference="right_wheel_link">
-        <material>Gazebo/Grey</material>
+    <gazebo reference="right_front_dif">
+        <material>Gazebo/Green</material>
     </gazebo>
-    <gazebo reference="left_wheel_link">
-        <material>Gazebo/Grey</material>
+    <gazebo reference="left_front_dif">
+        <material>Gazebo/Green</material>
     </gazebo>
-    <gazebo reference="caster_wheel_link">
-        <material>Gazebo/Grey</material>
-        <mu1 value="0.1"/> <!-- yumuşatmak için kullanılır.-->
-        <mu2 value="0.1"/>
+    <gazebo reference="right_front_wheel_link">
+        <material>Gazebo/Black</material>
     </gazebo>
+    <gazebo reference="left_front_wheel_link">
+        <material>Gazebo/Black</material>
+    </gazebo>
+    <gazebo reference="right_back_wheel_link">
+        <material>Gazebo/Black</material>
+    </gazebo>
+    <gazebo reference="left_back_wheel_link">
+        <material>Gazebo/Black</material>
+    </gazebo>
+    <!-- ACKERMANN DRİVE PLUGİN  -->
     <gazebo>
-    <plugin name="diff_drive_controller" filename="libgazebo_ros_diff_drive.so">
-      <!-- Update rate in Hz -->
-      <update_rate>50</update_rate>
-      <!-- wheels -->
-      <left_joint>base_left_wheel_joint</left_joint>
-      <right_joint>base_right_wheel_joint</right_joint>
-      <!-- kinematics -->
-      <wheel_separation>0.45</wheel_separation> <!-- base_witdh + tekerlik yüksekliği-->
-      <wheel_diameter>0.2</wheel_diameter> <!-- tekerlik radiusu-->
-      <!-- limits -->
-      <!-- <max_wheel_torque>20</max_wheel_torque>
-      <max_wheel_acceleration>1.0</max_wheel_acceleration> -->
-      <!-- input -->
-      <!-- <command_topic>cmd_vel</command_topic> -->
-      <!-- output -->
-      <publish_odom>true</publish_odom>
-      <publish_odom_tf>true</publish_odom_tf>
-      <publish_wheel_tf>true</publish_wheel_tf>
-      <odometry_topic>odom</odometry_topic>
-      <odometry_frame>odom</odometry_frame>
-      <robot_base_frame>base_footprint</robot_base_frame>
+        <plugin name="gazebo_ros_ackermann_drive" filename="libgazebo_ros_ackermann_drive.so">
+            <update_rate>100.0</update_rate>
+            <!-- wheels -->
+            <front_left_joint>left_front_dif_wheel_joint</front_left_joint>
+            <front_right_joint>right_front_dif_wheel_joint</front_right_joint>
+            <rear_left_joint>left_back_wheel_joint</rear_left_joint>
+            <rear_right_joint>right_back_wheel_joint</rear_right_joint>
+            <left_steering_joint>left_front_dif_joint</left_steering_joint>
+            <right_steering_joint>right_front_dif_joint </right_steering_joint>
+            <!-- <steering_wheel_joint>steering_wheel_joint</steering_wheel_joint> -->
+            <!-- Max absolute steer angle for tyre in radians-->
+            <!-- Any cmd_vel angular z greater than this would be capped -->
+            <max_steer>0.6458</max_steer>
+            <!-- Max absolute steering angle of steering wheel -->
+            <max_steering_angle>7.85</max_steering_angle>
+            <!-- Max absolute linear speed in m/s -->
+            <max_speed>20</max_speed>
+            <!-- PID tuning -->
+            <left_steering_pid_gain>1500 0 1</left_steering_pid_gain>
+            <left_steering_i_range>0 0</left_steering_i_range>
+            <right_steering_pid_gain>1500 0 1</right_steering_pid_gain>
+            <right_steering_i_range>0 0</right_steering_i_range>
+            <linear_velocity_pid_gain>1000 0 1</linear_velocity_pid_gain>
+            <linear_velocity_i_range>0 0</linear_velocity_i_range>
+            <!-- output -->
+            <publish_odom>true</publish_odom>
+            <publish_odom_tf>true</publish_odom_tf>
+            <publish_wheel_tf>true</publish_wheel_tf>
+            <publish_distance>true</publish_distance>
+            <publish_steerangle>true</publish_steerangle>
+            <odometry_frame>odom</odometry_frame>
+            <robot_base_frame>base_footprint</robot_base_frame>
     </plugin>
     </gazebo>

File: src/my_robot_description/urdf/my_robot.urdf.xacro (robot description, xacro)
@@ -4,5 +4,5 @@
     <xacro:include filename="mobile_base.xacro"/>
     <xacro:include filename="mobile_base_gazebo.xacro"/>
-    <xacro:include filename="robot_arm.xacro"/>
-    <xacro:include filename="robot_arm_gazebo.xacro"/>
+    <xacro:include filename="sensor.xacro"/>
+    <xacro:include filename="sensor_gazebo.xacro"/>
 </robot>
