Commit message: ackerman-project gps steering

File: src/my_robot_description/urdf/mobile_base.xacro (robot description, xacro)
@@ -26,5 +26,5 @@
             <origin xyz="0 0 ${base_height / 2.0}" rpy="0 0 0" />
         </collision>
-        <xacro:box_inertia m="5.0" l="${2*base_length}" w="${2*base_width}" h="${2*base_height}"
+        <xacro:box_inertia m="5" l="${base_height}" w="${base_length}" h="${base_width}"
                                 xyz="0 0 ${base_height / 2.0}" rpy="0 0 0" />
     </link>
@@ -66,5 +66,5 @@
                 <origin xyz="0 0 ${z_offset/2.0}" rpy="0 0 0" />
             </collision>
-            <xacro:cylinder_inertia m="1.0" r="${2*radius_}" l="${2*length_}"
+            <xacro:cylinder_inertia m="1.0" r="${2+radius_}" l="${2+length_}"
                     xyz="0 0 ${z_offset/2.0}" rpy="0 0 0" />
         </link>
@@ -74,26 +74,4 @@
     <xacro:wheel_link prefix="right_back" radius_="${wheel_radius}" length_="${wheel_length}"  z_offset="${wheel_length}"/>
     <xacro:wheel_link prefix="left_back" radius_="${wheel_radius}" length_="${wheel_length}" z_offset="${-wheel_length}"/>
-    <!-- <link name="steering_wheel_link">
-        <visual>
-            <geometry>
-                <cylinder length="0.05" radius="0.2"/>
-            </geometry>
-            <material name="grey"/>
-        </visual>
-        <collision>
-            <geometry>
-                <cylinder length="0.05" radius="0.2"/>
-            </geometry>
-        </collision>
-        <inertial>
-            <mass value="0.5"/>
-            <inertia ixx="0.001" ixy="0" ixz="0" iyy="0.001" iyz="0" izz="0.001"/>
-        </inertial>
-    </link> -->
-    <joint name="base_footprint_joint" type="fixed">
-        <parent link="odom"/>
-        <child link="base_footprint"/>
-        <origin rpy="0 0 0" xyz="0 0 0"/>
-    </joint>
     <joint name="base_joint" type="fixed">
         <parent link="base_footprint" />
@@ -145,10 +123,3 @@
         <limit effort="100" velocity="100"/>
     </joint>
-<!--
-    <joint name="steering_wheel_joint" type="continuous">
-        <parent link="base_link" />
-        <child link="steering_wheel_link" />
-        <origin xyz="0 0 0" rpy="0 0 0" />
-        <axis xyz="0 0 1" />
-    </joint> -->
 </robot>
